File: esp32/shortwave/sh0rtwave_pcb/sh0rtwave_pcb.kicad_sch (KiCad schematic)
At the start: 6 parts, among them J2 Conn_01x05, U1 XIAO_ESP32_S3, U2 AMPLIFIER

Commit message: pcb
Parts:
- added D1: LED, symbol Device:LED
- added R2: 330, symbol Device:R_US
- added R3: R_US, symbol Device:R_US
- added SW1: SW_Push, symbol Switch:SW_Push
Connections:
- net GND: now also R2.2, R3.2
- net at C1.1, R1.1, U1.12 (3V3)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: now also SW1.1
- net at U1.3 (D2/GPIO3): now also D1.2 (A)
- net at U1.4 (D3/GPIO4): now also U1.5 (D4/GPIO5), U1.6 (D5/GPIO6), R3.1, SW1.2
- new net: D1.1 (K), R2.1
Other:
- title: (none) -> sh0rtwave
- moved on the sheet: C1
