File: esp32/shortwave/sh0rtwave_pcb/sh0rtwave_pcb.kicad_pcb (KiCad board)
At the start: 2 copper layers, 11 parts

Commit message: pcb
Parts:
- removed 300: Resistor, Resistor_THT:R_Axial_DIN0207_L6.3mm_D2.5mm_P10.16mm_Horizontal
- removed 5v in: JST_PH_B2B-PH-K_1x02_P2.00mm_Vertical, Connector_JST:JST_PH_B2B-PH-K_1x02_P2.00mm_Vertical
- removed BUTTON: BUTTON, Connector_PinHeader_2.54mm:PinHeader_1x02_P2.54mm_Vertical
- added 330: R_Axial_DIN0207_L6.3mm_D2.5mm_P10.16mm_Horizontal, Resistor_THT:R_Axial_DIN0207_L6.3mm_D2.5mm_P10.16mm_Horizontal, F.Cu at (126.0, 65.9)
- added ?: , , F.Cu at (125.5, 52.0)
- added BTN: BTN, Connector_PinHeader_2.54mm:PinHeader_1x02_P2.54mm_Vertical, F.Cu at (90.0, 52.5)
- added PWR: 5v, Connector_JST:JST_PH_B2B-PH-K_1x02_P2.00mm_Vertical, F.Cu at (126.0, 95.5)
- added REF**: , MountingHole:MountingHole_3.2mm_M3, F.Cu at (83.5, 99.0)
- added REF**: , MountingHole:MountingHole_3.2mm_M3, F.Cu at (84.5, 52.5)
- 1k: value Resistor -> 1k
- moved 100uF 39.0 mm to (96.0, 69.0)
- moved 1k 13.7 mm to (83.9, 67.6), turned to 45 degrees
- moved LED 7.41 mm to (126.0, 58.5)
Routing:
- net (no net): track 760.5 -> 765.7 mm
Other:
- board text added: "sh0rtwave"

Commit message: pcb
Parts:
- moved REF** 1.41 mm to (84.5, 98.0)
Changed lines of the file:
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@@
 			(drillshape 0)
 			(scaleselection 1)
-			(outputdirectory "")
+			(outputdirectory "shortwave_pcb_2026-05-26/")
 		)
 	)
 	(footprint "MountingHole:MountingHole_3.2mm_M3"
 		(layer "F.Cu")
-		(at 83.5 99)
+		(at 84.5 98)
 		(descr "Mounting Hole 3.2mm, M3, no annular, generated by kicad-footprint-generator mountinghole.py")
 		(tags "mountinghole M3")

Commit message: share recordings
Other:
- board outline added: 51 x 57.5 mm
Changed lines of the file:
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@@
 			(drillshape 0)
 			(scaleselection 1)
-			(outputdirectory "shortwave_pcb_2026-05-26/")
+			(outputdirectory "shortwave_pcb_2026-05-31/")
 		)
 	)
@@
 		(layer "F.Cu")
 	)
+	(gr_rect
+		(start 80 47.5)
+		(end 131 105)
+		(stroke
+			(width 0.05)
+			(type default)
+		)
+		(fill no)
+		(layer "Edge.Cuts")
+	)
 	(gr_text "VDD\n"

Commit message: useSocket
Parts:
- removed ?: , 
- removed REF** (x2): , MountingHole:MountingHole_3.2mm_M3
- moved BTN 10.00 mm to (99.9, 53.8)
- moved INP441 8.90 mm to (100.0, 82.9)
- moved 100nF 8.90 mm to (93.5, 83.0)
- moved 1k 8.61 mm to (92.5, 67.0), turned to 90 degrees
- moved PWR 7.57 mm to (125.0, 88.0)
- moved MAX98357 7.51 mm to (112.0, 84.5)
- moved 10 4.61 mm to (93.5, 70.3)
- moved 100uF 3.54 mm to (96.5, 65.5)
- moved 330 2.00 mm to (124.0, 65.9)
- moved LED 2.00 mm to (124.0, 58.5)
- moved ESP32 S3 0.09 mm to (112.0, 61.9)
Routing:
- net (no net): track 765.7 -> 463.7 mm
Other:
- board size 51 x 57.5 mm -> 37.2 x 43.6 mm
- board text removed: "SV"
