File: esp32/shortwave/sh0rtwave_pcb/sh0rtwave_pcb.kicad_pcb (KiCad board)
At the start: 2 copper layers, 37.2 x 43.6 mm, 11 parts

Commit message: update schematic
Parts:
- 5v in: renamed from PWR
Changed lines of the file:
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@@
 			(drillshape 0)
 			(scaleselection 1)
-			(outputdirectory "shortwave_pcb_2026-05-31/")
+			(outputdirectory "shortwave_pcb_2026-06-12/")
 		)
 	)
@@
 		(tags "Through hole pin header THT 1x05 2.54mm single row")
 		(property "Reference" "INP441"
-			(at 0 -2.42 0)
+			(at 2 4.58 270)
 			(layer "F.SilkS")
 			(effects
@@
 		(tags "Resistor Axial_DIN0207 series Axial Horizontal pin pitch 10.16mm 0.25W = 1/4W length 6.3mm diameter 2.5mm")
 		(property "Reference" "10"
-			(at 5.16 -2.5 90)
+			(at 5.16 2.5 90)
 			(layer "F.SilkS")
 			(effects
@@
 		(descr "JST PH series connector, B2B-PH-K (http://www.jst-mfg.com/product/pdf/eng/ePH.pdf)")
 		(tags "connector JST PH vertical")
-		(property "Reference" "PWR"
-			(at -4 0.5 90)
+		(property "Reference" "5v in"
+			(at -3.5 0.5 0)
 			(layer "F.SilkS")
 			(effects
@@
 		(tags "C Disc series Radial pin pitch 5.00mm diameter 5mm width 2.5mm Capacitor")
 		(property "Reference" "100nF"
-			(at 8.5 1 90)
+			(at 2.5 2 90)
 			(layer "F.SilkS")
 			(effects
@@
 		)
 		(property "Value" "Capacitor"
-			(at 7.5 2.5 90)
-			(layer "F.Fab")
-			(effects
+			(at 8 -0.5 90)
+			(layer "F.Fab")
+			(effects
