File: esp32/shortwave/sh0rtwave_pcb/sh0rtwave_pcb.kicad_pcb (KiCad board)
At the start: 2 copper layers, 37.2 x 43.6 mm, 11 parts

Commit message: update glowstick, shortwave pcb
Routing:
- net (no net): track 463.7 -> 519.4 mm
Other:
- board size 37.2 x 43.6 mm -> 36.2 x 43.2 mm
