File: esp32/lightstick/Untitled/Untitled.kicad_pcb (KiCad board)
At the start: 2 copper layers, 40.5 x 26 mm, 10 parts, among them J1 Conn_02x09_Odd_Even, J2 Conn_01x04_Pin, J3 Conn_01x02_Pin, J4 Conn_01x02_Pin, Q1 S8050

Commit message: update shortwave firmware
Parts:
- GND OUT: renamed from J3
- renumbered R2 to 1k, J1 to 2272, R1 to 750k, J2 to RX, Q1 to S8050
